Commit message: Try to fix summit rotation

File: multirobots_ws/src/summit_xl_description/robots/summit_xl_std.urdf (robot description, URDF)
Before this commit: robot summit_xl, 22 links, 21 joints
Links:
- removed link summit_xl_front_ptz_camera_base_link
- removed link summit_xl_front_ptz_camera_frame_link
- removed link summit_xl_front_ptz_camera_optical_frame_link
- removed link summit_xl_front_ptz_camera_pan_link
- removed link summit_xl_front_ptz_camera_tilt_link
- removed link summit_xl_front_rgbd_camera_depth_frame
- removed link summit_xl_front_rgbd_camera_depth_optical_frame
- removed link summit_xl_front_rgbd_camera_link
- removed link summit_xl_front_rgbd_camera_rgb_frame
- removed link summit_xl_front_rgbd_camera_rgb_optical_frame
- removed link summit_xl_gps_base_link
- removed link summit_xl_gps_mast_base_link
- removed link summit_xl_imu_link
- link summit_xl_front_laser_base_link: mass 0.130 -> 0.190; geometry collision mesh filename=package://robotnik_sensors/meshes/lidar_m10_p.STL; visual mesh filename=package://robotnik_sensors/meshes/lidar_m10_p.STL
Joints:
- removed joint summit_xl_front_ptz_camera_frame_joint
- removed joint summit_xl_front_ptz_camera_joint
- removed joint summit_xl_front_ptz_camera_optical_joint
- removed joint summit_xl_front_ptz_camera_pan_joint
- removed joint summit_xl_front_ptz_camera_tilt_joint
- removed joint summit_xl_front_rgbd_camera_depth_joint
- removed joint summit_xl_front_rgbd_camera_depth_optical_joint
- removed joint summit_xl_front_rgbd_camera_joint
- removed joint summit_xl_front_rgbd_camera_rgb_joint
- removed joint summit_xl_front_rgbd_camera_rgb_optical_joint
- removed joint summit_xl_gps_joint
- removed joint summit_xl_gps_mast_joint
- removed joint summit_xl_imu_joint
- joint summit_xl_front_laser_joint: origin xyz=0.00 0.0 0.0474 rpy=0 0 0 -> xyz=0.05 0.05 0.05 rpy=0 0 0

File: multirobots_ws/src/summit_xl_description/urdf/wheels/rubber_wheel.urdf.xacro (robot description, xacro)
@@ -67,10 +67,18 @@
      </transmission>
     <gazebo reference="${prefix}_wheel">
-			<mu1 value="1.0"/>
-			<mu2 value="1.0"/>
-			<kp value="10000000.0" />
-			<kd value="1.0" />
-			<fdir1 value="1 0 0"/>
-      <turnGravityOff>false</turnGravityOff>
+      <!-- <collision>
+        <surface>
+          <friction>
+            <ode> -->
+              <mu1 value="1.0"/>
+              <mu2 value="1.0"/>
+              <kp value="10000000.0" />
+              <kd value="1.0" />
+              <fdir1 value="1 0 0"/>
+              <turnGravityOff>false</turnGravityOff>
+            <!-- </ode>
+          </friction>
+        </surface>
+      </collision> -->
     </gazebo>
   </xacro:macro>

Commit message: Add IMU sensor & rosbag

File: multirobots_ws/src/summit_xl_description/robots/summit_xl_std.urdf (robot description, URDF)
Before this commit: robot summit_xl, 9 links, 8 joints
Links:
- link summit_xl_front_laser_base_link: mass 0.190 -> 0.160; geometry visual mesh filename=package://robotnik_sensors/meshes/hokuyo_urg_04lx.dae
Joints:
- joint summit_xl_front_laser_joint: origin xyz=0.05 0.05 0.05 rpy=0 0 0 -> xyz=0.00 0 0.05315 rpy=0 0 0

File: multirobots_ws/src/summit_xl_description/robots/summit_xl_std.urdf.xacro (robot description, xacro)
@@ -66,8 +66,4 @@
 			<origin xyz="-0.18 0.0 0.170" rpy="0 0 0"/>
 		</xacro:sensor_imu-->
-		<!-- 2d laser >
-		<xacro:sensor_hokuyo_ust20lx prefix="$(arg prefix)front_laser" parent="$(arg prefix)base_link" prefix_topic="front_laser" gpu="$(arg gpu)">
-			<origin xyz="0.0 0.0 0.2726" rpy="0 0 0"/>
-		</xacro:sensor_hokuyo_ust20lx-->
 		<!-- ptz camera >
 		<xacro:sensor_axis prefix="$(arg prefix)front_ptz_camera" parent="$(arg prefix)base_link">
@@ -82,8 +78,12 @@
 			<origin xyz="-0.22 0 0.275" rpy="0 0 0"/>
 		</xacro:sensor_gps_with_mast-->
-		<!-- 2d laser -->
-		<xacro:sensor_lidar_m10_p id="$(arg id)" prefix="$(arg prefix)" prefix_laser="$(arg prefix)front_laser" parent="$(arg prefix)base_link">
+		<!-- IMU -->
+		<xacro:sensor_pixhawk id="$(arg id)" frame_prefix="$(arg prefix)imu_" name_prefix="$(arg prefix)" parent="$(arg prefix)base_link">
+			<origin xyz="-0.18 0.0 0.170" rpy="0 0 0"/>
+		</xacro:sensor_pixhawk>
+		<!-- 2d lidar -->
+		<xacro:sensor_hokuyo_urg04lx id="$(arg id)" frame_prefix="$(arg prefix)front_laser_" name_prefix="$(arg prefix)" parent="$(arg prefix)base_link">
 			<origin xyz="0.0 0.0 0.2726" rpy="0 0 0"/>
-		</xacro:sensor_lidar_m10_p>
+		</xacro:sensor_hokuyo_urg04lx>
    </xacro:macro>
    <!-- Gazebo ros control pluggins -->
