Commit message: Use of xacro files & ros_gz_bridge

File: multirobots_ws/src/summit_xl_description/robots/summit_xl_std.urdf.xacro (robot description, xacro)
@@ -9,5 +9,5 @@
 	<!-- Import summit XL wheels -->
 	<xacro:include filename="$(find summit_xl_description)/urdf/wheels/rubber_wheel.urdf.xacro" />
-  <xacro:include filename="$(find summit_xl_description)/urdf/wheels/omni_wheel.urdf.xacro" />
+  	<xacro:include filename="$(find summit_xl_description)/urdf/wheels/omni_wheel.urdf.xacro" />
 	<!-- Import all available sensors -->
 	<xacro:include filename="$(find robotnik_sensors)/urdf/all_sensors.urdf.xacro" />
@@ -21,5 +21,5 @@
 	<xacro:arg name="prefix" default="summit_xl_"/>
 	<xacro:arg name="ros_planar_move_plugin" default="false"/>
-  <xacro:arg name="ros_planar_move_plugin_force_based" default="false"/>
+  	<xacro:arg name="ros_planar_move_plugin_force_based" default="false"/>
 	<xacro:arg name="omni_wheels" default="false"/>
 	<xacro:arg name="gpu" default="false"/>
@@ -33,52 +33,56 @@
 		<!-- Summit XL base -->
 		<xacro:summit_xl_base prefix="$(arg prefix)" publish_bf="true" hq="${hq}" />
-    <xacro:unless value="$(arg omni_wheels)">
-  		<xacro:rubber_wheel prefix="$(arg prefix)front_right" parent="$(arg prefix)base_link" reflect="false" hq="${hq}">
-  			<origin xyz="${wheel_offset_x} -${wheel_offset_y} ${wheel_offset_z}" rpy="0 0 0"/>
-  		</xacro:rubber_wheel>
-  		<xacro:rubber_wheel prefix="$(arg prefix)front_left" parent="$(arg prefix)base_link" reflect="true" hq="${hq}">
-  			<origin xyz="${wheel_offset_x} ${wheel_offset_y} ${wheel_offset_z}" rpy="0 0 0"/>
-  		</xacro:rubber_wheel>
-  		<xacro:rubber_wheel prefix="$(arg prefix)back_left" parent="$(arg prefix)base_link" reflect="true" hq="${hq}">
-  			<origin xyz="-${wheel_offset_x} ${wheel_offset_y} ${wheel_offset_z}" rpy="0 0 0"/>
-  		</xacro:rubber_wheel>
-  		<xacro:rubber_wheel prefix="$(arg prefix)back_right" parent="$(arg prefix)base_link" reflect="false" hq="${hq}">
-  			<origin xyz="-${wheel_offset_x} -${wheel_offset_y} ${wheel_offset_z}" rpy="0 0 0"/>
-  		</xacro:rubber_wheel>
-    </xacro:unless>
-    <xacro:if value="$(arg omni_wheels)">
-  		<xacro:omni_wheel prefix="$(arg prefix)front_right" parent="$(arg prefix)base_link" reflect="false" hq="${hq}">
-  			<origin xyz="${wheel_offset_x} -${wheel_offset_y} ${wheel_offset_z}" rpy="0 0 0"/>
-  		</xacro:omni_wheel>
-  		<xacro:omni_wheel prefix="$(arg prefix)front_left" parent="$(arg prefix)base_link" reflect="true" hq="${hq}">
-  			<origin xyz="${wheel_offset_x} ${wheel_offset_y} ${wheel_offset_z}" rpy="0 0 0"/>
-  		</xacro:omni_wheel>
-  		<xacro:omni_wheel prefix="$(arg prefix)back_left" parent="$(arg prefix)base_link" reflect="true" hq="${hq}">
-  			<origin xyz="-${wheel_offset_x} ${wheel_offset_y} ${wheel_offset_z}" rpy="0 0 0"/>
-  		</xacro:omni_wheel>
-  		<xacro:omni_wheel prefix="$(arg prefix)back_right" parent="$(arg prefix)base_link" reflect="false" hq="${hq}">
-  			<origin xyz="-${wheel_offset_x} -${wheel_offset_y} ${wheel_offset_z}" rpy="0 0 0"/>
-  		</xacro:omni_wheel>
-    </xacro:if>
-        <!-- IMU -->
+		<xacro:unless value="$(arg omni_wheels)">
+			<xacro:rubber_wheel prefix="$(arg prefix)front_right" parent="$(arg prefix)base_link" reflect="false" hq="${hq}">
+				<origin xyz="${wheel_offset_x} -${wheel_offset_y} ${wheel_offset_z}" rpy="0 0 0"/>
+			</xacro:rubber_wheel>
+			<xacro:rubber_wheel prefix="$(arg prefix)front_left" parent="$(arg prefix)base_link" reflect="true" hq="${hq}">
+				<origin xyz="${wheel_offset_x} ${wheel_offset_y} ${wheel_offset_z}" rpy="0 0 0"/>
+			</xacro:rubber_wheel>
+			<xacro:rubber_wheel prefix="$(arg prefix)back_left" parent="$(arg prefix)base_link" reflect="true" hq="${hq}">
+				<origin xyz="-${wheel_offset_x} ${wheel_offset_y} ${wheel_offset_z}" rpy="0 0 0"/>
+			</xacro:rubber_wheel>
+			<xacro:rubber_wheel prefix="$(arg prefix)back_right" parent="$(arg prefix)base_link" reflect="false" hq="${hq}">
+				<origin xyz="-${wheel_offset_x} -${wheel_offset_y} ${wheel_offset_z}" rpy="0 0 0"/>
+			</xacro:rubber_wheel>
+		</xacro:unless>
+		<xacro:if value="$(arg omni_wheels)">
+			<xacro:omni_wheel prefix="$(arg prefix)front_right" parent="$(arg prefix)base_link" reflect="false" hq="${hq}">
+				<origin xyz="${wheel_offset_x} -${wheel_offset_y} ${wheel_offset_z}" rpy="0 0 0"/>
+			</xacro:omni_wheel>
+			<xacro:omni_wheel prefix="$(arg prefix)front_left" parent="$(arg prefix)base_link" reflect="true" hq="${hq}">
+				<origin xyz="${wheel_offset_x} ${wheel_offset_y} ${wheel_offset_z}" rpy="0 0 0"/>
+			</xacro:omni_wheel>
+			<xacro:omni_wheel prefix="$(arg prefix)back_left" parent="$(arg prefix)base_link" reflect="true" hq="${hq}">
+				<origin xyz="-${wheel_offset_x} ${wheel_offset_y} ${wheel_offset_z}" rpy="0 0 0"/>
+			</xacro:omni_wheel>
+			<xacro:omni_wheel prefix="$(arg prefix)back_right" parent="$(arg prefix)base_link" reflect="false" hq="${hq}">
+				<origin xyz="-${wheel_offset_x} -${wheel_offset_y} ${wheel_offset_z}" rpy="0 0 0"/>
+			</xacro:omni_wheel>
+		</xacro:if>
+        <!-- IMU >
 		<xacro:sensor_imu prefix="$(arg prefix)imu" parent="$(arg prefix)base_link" topic="imu/data_raw">
 			<origin xyz="-0.18 0.0 0.170" rpy="0 0 0"/>
-		</xacro:sensor_imu>
-		<!-- 2d laser -->
+		</xacro:sensor_imu-->
+		<!-- 2d laser >
 		<xacro:sensor_hokuyo_ust20lx prefix="$(arg prefix)front_laser" parent="$(arg prefix)base_link" prefix_topic="front_laser" gpu="$(arg gpu)">
 			<origin xyz="0.0 0.0 0.2726" rpy="0 0 0"/>
-		</xacro:sensor_hokuyo_ust20lx>
-		<!-- ptz camera -->
+		</xacro:sensor_hokuyo_ust20lx-->
+		<!-- ptz camera >
 		<xacro:sensor_axis prefix="$(arg prefix)front_ptz_camera" parent="$(arg prefix)base_link">
 			<origin xyz="0.185 0 0.1967" rpy="0 ${15*PI/180} 0"/>
-		</xacro:sensor_axis>
-	  <!-- RGBD -->
+		</xacro:sensor_axis-->
+	  <!-- RGBD >
 	  <xacro:sensor_orbbec_astra prefix="$(arg prefix)front_rgbd_camera" parent="$(arg prefix)base_link" prefix_topic="front_rgbd_camera">
 			<origin xyz="0.324 0.012 0.172" rpy="0 0 0"/>
-		</xacro:sensor_orbbec_astra>
-	  <!-- GPS -->
+		</xacro:sensor_orbbec_astra-->
+	  <!-- GPS >
 	  <xacro:sensor_gps_with_mast prefix="$(arg prefix)gps" parent="$(arg prefix)base_link" gps_latitude="$(arg gps_latitude)" gps_longitude="$(arg gps_longitude)">
 			<origin xyz="-0.22 0 0.275" rpy="0 0 0"/>
-		</xacro:sensor_gps_with_mast>
+		</xacro:sensor_gps_with_mast-->
+		<!-- 2d laser -->
+		<xacro:sensor_lidar_m10_p prefix="$(arg prefix)front_laser" parent="$(arg prefix)base_link" prefix_topic="front_laser" gpu="$(arg gpu)">
+			<origin xyz="0.0 0.0 0.2726" rpy="0 0 0"/>
+		</xacro:sensor_lidar_m10_p>
    </xacro:macro>
    <!-- Gazebo ros control pluggins -->

File: multirobots_ws/src/summit_xl_description/urdf/bases/summit_xl_base.gazebo.xacro (robot description, xacro)
@@ -1,117 +1,53 @@
 <?xml version="1.0"?>
 <robot xmlns:xacro="http://wiki.ros.org/xacro">
-  <!-- ros control plugin -->
-  <xacro:macro name="ros_control">
-    <gazebo>
-      <plugin filename="libgz_ros2_control-system.so" name="gz_ros2_control">
-		<robotParam>robot_description</robotParam>
-        <controlPeriod>0.001</controlPeriod>
-	    <robotSimType>gazebo_ros_control/DefaultRobotHWSim</robotSimType>
-		<legacyModeNS>true</legacyModeNS>
-      </plugin>
-    </gazebo>
+	<!-- ros2 control plugin -->
+	<xacro:macro name="ros_control">
+		<ros2_control name="GazeboSimSystem" type="system">
+			<hardware>
+				<plugin>gz_ros2_control/GazeboSimSystem</plugin>
+			</hardware>
+			<joint name="summit_xl_front_left_wheel_joint">
+				<command_interface name="velocity">
+					<param name="min">-10</param>
+					<param name="max">10</param>
+				</command_interface>
+				<state_interface name="position"/>
+				<state_interface name="velocity"/>
+			</joint>
+			<joint name="summit_xl_front_right_wheel_joint">
+				<command_interface name="velocity">
+					<param name="min">-10</param>
+					<param name="max">10</param>
+				</command_interface>
+				<state_interface name="position"/>
+				<state_interface name="velocity"/>
+			</joint>
+			<joint name="summit_xl_back_left_wheel_joint">
+				<command_interface name="velocity">
+					<param name="min">-10</param>
+					<param name="max">10</param>
+				</command_interface>
+				<state_interface name="position"/>
+				<state_interface name="velocity"/>
+			</joint>
+			<joint name="summit_xl_back_right_wheel_joint">
+				<command_interface name="velocity">
+					<param name="min">-10</param>
+					<param name="max">10</param>
+				</command_interface>
+				<state_interface name="position"/>
+				<state_interface name="velocity"/>
+			</joint>
+		</ros2_control>
+		<gazebo>
+			<plugin filename="libgz_ros2_control-system.so" name="gz_ros2_control::GazeboSimROS2ControlPlugin">
+				<robot_param>robot_description</robot_param>
+				<robot_param_node>robot_state_publisher</robot_param_node>
+				<parameters>/home/multirobots/multirobots_ws/install/summit_xl_description/share/summit_xl_description/config/summit_control.yaml</parameters>
+			</plugin>
+		</gazebo>
 	</xacro:macro>
-	<!-- skid steering plugin -->
-	<xacro:macro name="skid_steering" params="prefix publish_tf">
-    <gazebo>
-      <plugin name="skid_steer_drive_controller" filename="libgazebo_ros_skid_steer_drive.so">
-			<!--<robotNamespace>/summit_xl</robotNamespace>-->
-		    <updateRate>50.0</updateRate>
-		    <leftFrontJoint>${prefix}front_left_wheel_joint</leftFrontJoint>
-		    <rightFrontJoint>${prefix}front_right_wheel_joint</rightFrontJoint>
-		    <leftRearJoint>${prefix}back_left_wheel_joint</leftRearJoint>
-		    <rightRearJoint>${prefix}back_right_wheel_joint</rightRearJoint>
-		    <!-- wheelSeparation>0.566</wheelSeparation --> <!-- real parameter value -->
-		    <wheelSeparation>0.462</wheelSeparation> <!-- works a bit better in Gazebo -->
-		    <wheelDiameter>0.22</wheelDiameter>
-		    <robotBaseFrame>${prefix}base_footprint</robotBaseFrame>
-		    <torque>50</torque>
-		    <commandTopic>robotnik_base_control/cmd_vel</commandTopic>
-		    <odometryTopic>robotnik_base_control/odom</odometryTopic>
-		    <odometryFrame>${prefix}odom</odometryFrame>
-		    <broadcastTF>${publish_tf}</broadcastTF>
-      </plugin>
-    </gazebo>
-  </xacro:macro>
-  <xacro:macro name="omni_steering" params="prefix publish_tf force_based:=false">
-		<xacro:if value="${force_based}">
-			<gazebo>
-				<plugin name="ros_force_based_move" filename="librobotnik_force_based_move.so">
-					<commandTopic>robotnik_base_control/cmd_vel</commandTopic>
-					<odometryTopic>robotnik_base_control/odom</odometryTopic>
-					<odometryFrame>${prefix}odom</odometryFrame>
-					<yaw_velocity_p_gain>10000.0</yaw_velocity_p_gain>
-					<x_velocity_p_gain>10000.0</x_velocity_p_gain>
-					<y_velocity_p_gain>10000.0</y_velocity_p_gain>
-					<robotBaseFrame>${prefix}base_footprint</robotBaseFrame>
-					<commandWatchdog>1</commandWatchdog>
-					<odometryRate>50.0</odometryRate>
-					<publishOdometryTf>${publish_tf}</publishOdometryTf>
-				</plugin>
-			</gazebo>
-		</xacro:if>
-		<xacro:unless value="${force_based}">
-			<gazebo>
-				<plugin name="omni_steering" filename="libgazebo_ros_planar_move.so">
-				<commandTopic>robotnik_base_control/cmd_vel</commandTopic>
-				<odometryTopic>robotnik_base_control/odom</odometryTopic>
-				<odometryFrame>${prefix}odom</odometryFrame>
-				<odometryRate>50.0</odometryRate>
-				<robotBaseFrame>${prefix}base_footprint</robotBaseFrame>
-				<publishTF>${publish_tf}</publishTF>
-				<enableYAxis>true</enableYAxis>
-				</plugin>
-			</gazebo>
-		</xacro:unless>
-  </xacro:macro>
-  	<xacro:macro name="skid_steering" params="prefix publish_tf force_based">
-		<xacro:if value="${force_based}">
-			<gazebo>
-				<plugin name="ros_force_based_move" filename="librobotnik_force_based_move.so">
-					<commandTopic>robotnik_base_control/cmd_vel</commandTopic>
-					<odometryTopic>robotnik_base_control/odom</odometryTopic>
-					<odometryFrame>${prefix}odom</odometryFrame>
-					<yaw_velocity_p_gain>10000.0</yaw_velocity_p_gain>
-					<x_velocity_p_gain>10000.0</x_velocity_p_gain>
-					<y_velocity_p_gain>0.0</y_velocity_p_gain>
-					<robotBaseFrame>${prefix}base_footprint</robotBaseFrame>
-					<commandWatchdog>1</commandWatchdog>
-					<odometryRate>50.0</odometryRate>
-					<publishOdometryTf>${publish_tf}</publishOdometryTf>
-				</plugin>
-			</gazebo>
-		</xacro:if>
-	  	<xacro:unless value="${force_based}">
-			<gazebo>
-				<plugin name="skid_steering" filename="libgazebo_ros_planar_move.so">
-				<commandTopic>robotnik_base_control/cmd_vel</commandTopic>
-				<odometryTopic>robotnik_base_control/odom</odometryTopic>
-				<odometryFrame>${prefix}odom</odometryFrame>
-				<odometryRate>50.0</odometryRate>
-				<robotBaseFrame>${prefix}base_footprint</robotBaseFrame>
-				<publishTF>${publish_tf}</publishTF>
-				<enableYAxis>false</enableYAxis>
-				</plugin>
-			</gazebo>
-		</xacro:unless>
-  	</xacro:macro>
-  <xacro:macro name="ros_force_based_move" params="publish_tf prefix">
-	  <gazebo>
-		 <plugin name="ros_force_based_move" filename="librobotnik_force_based_move.so">
-			 <commandTopic>robotnik_base_control/cmd_vel</commandTopic>
-			 <odometryTopic>robotnik_base_control/odom</odometryTopic>
-	         <odometryFrame>${prefix}odom</odometryFrame>
-			 <yaw_velocity_p_gain>10000.0</yaw_velocity_p_gain>
-			 <x_velocity_p_gain>10000.0</x_velocity_p_gain>
-			 <y_velocity_p_gain>10000.0</y_velocity_p_gain>
-			 <robotBaseFrame>${prefix}base_footprint</robotBaseFrame>
-			 <commandWatchdog>1</commandWatchdog>
-			 <odometryRate>50.0</odometryRate>
-			 <publishOdometryTf>${publish_tf}</publishOdometryTf>
-		 </plugin>
-	  </gazebo>
-  </xacro:macro>
-  <gazebo reference="base_footprint">
-    <material>Gazebo/Green</material>
-  </gazebo>
+	<gazebo reference="base_footprint">
+		<material>Gazebo/Green</material>
+	</gazebo>
 </robot>

Commit message: Trying to spawn multiple summits (in comments)

File: multirobots_ws/src/summit_xl_description/robots/summit_xl_std.urdf.xacro (robot description, xacro)
@@ -26,4 +26,5 @@
 	<xacro:arg name="gps_latitude" default="0"/>
 	<xacro:arg name="gps_longitude" default="0"/>
+	<xacro:arg name="robot_namespace" default=""/>
     <xacro:macro name="summit_xl" params="prefix publish_bf hq">
 		<!-- *************** -->
@@ -87,5 +88,5 @@
    </xacro:macro>
    <!-- Gazebo ros control pluggins -->
-   <xacro:ros_control/>
+   <xacro:ros_control robot_namespace="$(arg robot_namespace)"/>
 	<xacro:if value="$(arg ros_planar_move_plugin)">
 		<xacro:if value="$(arg omni_wheels)">

File: multirobots_ws/src/summit_xl_description/urdf/bases/summit_xl_base.gazebo.xacro (robot description, xacro)
@@ -2,5 +2,5 @@
 <robot xmlns:xacro="http://wiki.ros.org/xacro">
 	<!-- ros2 control plugin -->
-	<xacro:macro name="ros_control">
+	<xacro:macro name="ros_control" params="robot_namespace">
 		<ros2_control name="GazeboSimSystem" type="system">
 			<hardware>
@@ -42,4 +42,6 @@
 		<gazebo>
 			<plugin filename="libgz_ros2_control-system.so" name="gz_ros2_control::GazeboSimROS2ControlPlugin">
+				<!-- <robot_param>${robot_namespace}/robot_description</robot_param>
+				<robot_param_node>${robot_namespace}/robot_state_publisher</robot_param_node> -->
 				<robot_param>robot_description</robot_param>
 				<robot_param_node>robot_state_publisher</robot_param_node>

Commit message: Debug lidar sensor

File: multirobots_ws/src/summit_xl_description/robots/summit_xl_std.urdf.xacro (robot description, xacro)
@@ -26,5 +26,5 @@
 	<xacro:arg name="gps_latitude" default="0"/>
 	<xacro:arg name="gps_longitude" default="0"/>
-	<xacro:arg name="robot_namespace" default="summit_xl_1"/>
+	<xacro:arg name="id" default="1"/>
     <xacro:macro name="summit_xl" params="prefix publish_bf hq">
 		<!-- *************** -->
@@ -83,10 +83,10 @@
 		</xacro:sensor_gps_with_mast-->
 		<!-- 2d laser -->
-		<xacro:sensor_lidar_m10_p prefix="$(arg prefix)front_laser" parent="$(arg prefix)base_link" prefix_topic="front_laser" gpu="$(arg gpu)">
+		<xacro:sensor_lidar_m10_p id="$(arg id)" prefix="$(arg prefix)" prefix_laser="$(arg prefix)front_laser" parent="$(arg prefix)base_link">
 			<origin xyz="0.0 0.0 0.2726" rpy="0 0 0"/>
 		</xacro:sensor_lidar_m10_p>
    </xacro:macro>
    <!-- Gazebo ros control pluggins -->
-   <xacro:ros_control robot_namespace="$(arg robot_namespace)"/>
+   <xacro:ros_control id="$(arg id)" prefix="$(arg prefix)"/>
 	<xacro:if value="$(arg ros_planar_move_plugin)">
 		<xacro:if value="$(arg omni_wheels)">

File: multirobots_ws/src/summit_xl_description/urdf/bases/summit_xl_base.gazebo.xacro (robot description, xacro)
@@ -2,5 +2,5 @@
 <robot xmlns:xacro="http://wiki.ros.org/xacro">
 	<!-- ros2 control plugin -->
-	<xacro:macro name="ros_control" params="robot_namespace">
+	<xacro:macro name="ros_control" params="id prefix">
 		<ros2_control name="GazeboSimSystem" type="system">
 			<hardware>
@@ -44,8 +44,8 @@
 				<robot_param>robot_description</robot_param>
 				<robot_param_node>robot_state_publisher</robot_param_node>
-				<parameters>/tmp/${robot_namespace}_control.yaml</parameters>
+				<parameters>/tmp/${prefix}${id}_control.yaml</parameters>
 				<!-- <controller_manager_name>controller_manager</controller_manager_name> -->
 				<ros>
-					<namespace>${robot_namespace}</namespace>
+					<namespace>${prefix}${id}</namespace>
 				</ros>
 			</plugin>

Commit message: Add gps & camera sensors

File: multirobots_ws/src/summit_xl_description/robots/summit_xl_std.urdf.xacro (robot description, xacro)
@@ -62,20 +62,8 @@
 			</xacro:omni_wheel>
 		</xacro:if>
-        <!-- IMU >
-		<xacro:sensor_imu prefix="$(arg prefix)imu" parent="$(arg prefix)base_link" topic="imu/data_raw">
-			<origin xyz="-0.18 0.0 0.170" rpy="0 0 0"/>
-		</xacro:sensor_imu-->
-		<!-- ptz camera >
-		<xacro:sensor_axis prefix="$(arg prefix)front_ptz_camera" parent="$(arg prefix)base_link">
-			<origin xyz="0.185 0 0.1967" rpy="0 ${15*PI/180} 0"/>
-		</xacro:sensor_axis-->
 	  <!-- RGBD >
 	  <xacro:sensor_orbbec_astra prefix="$(arg prefix)front_rgbd_camera" parent="$(arg prefix)base_link" prefix_topic="front_rgbd_camera">
 			<origin xyz="0.324 0.012 0.172" rpy="0 0 0"/>
 		</xacro:sensor_orbbec_astra-->
-	  <!-- GPS >
-	  <xacro:sensor_gps_with_mast prefix="$(arg prefix)gps" parent="$(arg prefix)base_link" gps_latitude="$(arg gps_latitude)" gps_longitude="$(arg gps_longitude)">
-			<origin xyz="-0.22 0 0.275" rpy="0 0 0"/>
-		</xacro:sensor_gps_with_mast-->
 		<!-- IMU -->
 		<xacro:sensor_pixhawk id="$(arg id)" frame_prefix="$(arg prefix)imu_" name_prefix="$(arg prefix)" parent="$(arg prefix)base_link">
@@ -86,4 +74,12 @@
 			<origin xyz="0.0 0.0 0.2726" rpy="0 0 0"/>
 		</xacro:sensor_hokuyo_urg04lx>
+		<!-- GPS -->
+	  	<xacro:sensor_gps id="$(arg id)" frame_prefix="$(arg prefix)gps_" name_prefix="$(arg prefix)" parent="$(arg prefix)base_link">
+			<origin xyz="-0.22 0 0.275" rpy="0 0 0"/>
+		</xacro:sensor_gps>
+		<!-- ptz camera -->
+		<xacro:sensor_axis_m5013 id="$(arg id)" frame_prefix="$(arg prefix)camera_" name_prefix="$(arg prefix)" parent="$(arg prefix)base_link">
+			<origin xyz="0.185 0 0.1967" rpy="0 ${15*PI/180} 0"/>
+		</xacro:sensor_axis_m5013>
    </xacro:macro>
    <!-- Gazebo ros control pluggins -->

Commit message: Add depth cameras & fix some sensors position

File: multirobots_ws/src/summit_xl_description/robots/summit_xl_std.urdf.xacro (robot description, xacro)
@@ -62,8 +62,4 @@
 			</xacro:omni_wheel>
 		</xacro:if>
-	  <!-- RGBD >
-	  <xacro:sensor_orbbec_astra prefix="$(arg prefix)front_rgbd_camera" parent="$(arg prefix)base_link" prefix_topic="front_rgbd_camera">
-			<origin xyz="0.324 0.012 0.172" rpy="0 0 0"/>
-		</xacro:sensor_orbbec_astra-->
 		<!-- IMU -->
 		<xacro:sensor_pixhawk id="$(arg id)" frame_prefix="$(arg prefix)imu_" name_prefix="$(arg prefix)" parent="$(arg prefix)base_link">
@@ -80,6 +76,12 @@
 		<!-- ptz camera -->
 		<xacro:sensor_axis_m5013 id="$(arg id)" frame_prefix="$(arg prefix)camera_" name_prefix="$(arg prefix)" parent="$(arg prefix)base_link">
-			<origin xyz="0.185 0 0.1967" rpy="0 ${15*PI/180} 0"/>
+			<!-- <origin xyz="0.185 0 0.1967" rpy="0 ${15*PI/180} 0"/> -->
+			<origin xyz="0.185 0 0.23" rpy="0 ${-75*PI/180} 0"/>
 		</xacro:sensor_axis_m5013>
+		<!-- depth camera -->
+		<xacro:sensor_azure_kinect id="$(arg id)" frame_prefix="$(arg prefix)depth_camera_" name_prefix="$(arg prefix)" parent="$(arg prefix)base_link">
+			<!-- <origin xyz="0.324 0.012 0.172" rpy="0 0 ${PI/2}"/> -->
+			<origin xyz="0.324 0.012 0.172" rpy="0 0 ${PI/2}"/>
+		</xacro:sensor_azure_kinect>
    </xacro:macro>
    <!-- Gazebo ros control pluggins -->
