Commit message: Rm squashfs-root from github & minor fixes

File: multirobots_ws/src/summit_xl_description/urdf/bases/summit_xl_base.gazebo.xacro (robot description, xacro)
@@ -39,4 +39,22 @@
 				<state_interface name="velocity"/>
 			</joint>
+			<joint name="summit_xl_camera_pan_joint">
+				<command_interface name="position">
+					<param name="min">-3.1416</param>
+					<param name="max">3.1416</param>
+				</command_interface>
+				<state_interface name="position"/>
+				<state_interface name="velocity"/>
+				<state_interface name="effort"/>
+			</joint>
+			<joint name="summit_xl_camera_tilt_joint">
+				<command_interface name="position">
+					<param name="min">-1.5708</param>
+					<param name="max">1.5708</param>
+				</command_interface>
+				<state_interface name="position"/>
+				<state_interface name="velocity"/>
+				<state_interface name="effort"/>
+			</joint>
 		</ros2_control>
 		<gazebo>
