Commit message: Fix textures & system plugins

File: multirobots_ws/src/summit_xl_description/urdf/bases/summit_xl_base.urdf.xacro (robot description, xacro)
@@ -41,7 +41,7 @@
 		   </geometry>
 		   </xacro:unless>
-		   <material name="darkgrey">
+		   <!-- <material name="darkgrey">
 			 <color rgba="0.1 0.1 0.1 1"/>
-		   </material>
+		   </material> -->
 		</visual>
 		<collision>
