Commit message: Minor fixes & notes added

File: multirobots_ws/src/summit_xl_description/urdf/wheels/rubber_wheel.urdf.xacro (robot description, xacro)
@@ -67,18 +67,10 @@
      </transmission>
     <gazebo reference="${prefix}_wheel">
-      <!-- <collision>
-        <surface>
-          <friction>
-            <ode> -->
-              <mu1 value="1.0"/>
-              <mu2 value="0.8"/>
-              <kp value="10000000.0" />
-              <kd value="1.0" />
-              <fdir1 value="1 0 0"/>
-              <turnGravityOff>false</turnGravityOff>
-            <!-- </ode>
-          </friction>
-        </surface>
-      </collision> -->
+      <mu1 value="1.0"/>
+      <mu2 value="0.7"/>
+      <kp value="10000000.0" />
+      <kd value="1.0" />
+      <fdir1 value="1 0 0"/>
+      <turnGravityOff>false</turnGravityOff>
     </gazebo>
   </xacro:macro>
